Commit message: added basic urdf robot and launch file

File: mechanical_ws/urdf_robot/urdf/my_robot.urdf (robot description, URDF)
Before this commit: robot GuilleBot, 16 links, 15 joints
Links:
- link left_gripper: geometry visual cylinder length=0.2 radius=0.01
- link left_tip: geometry visual cylinder length=0.2 radius=0.01
- link right_gripper: geometry visual cylinder length=0.2 radius=0.01
- link right_tip: geometry visual cylinder length=0.2 radius=0.01
